File: rootpad/rootpad.kicad_pcb (KiCad board)
At the start: 2 copper layers, 77.8 x 110.3 mm, 56 parts, among them J1 USB_B_Mini, SW1 SW_Push, U1 ATmega32U4-AU, Y1 16MHz

Commit message: Connected diodes and reset
Parts:
- D1, D10, D11, D12, D13, D14, D15, D16, D17, D18, D2, D3, D4, D5, D6, D7, D8, D9: footprint Diode_THT:D_DO-35_SOD27_P7.62mm_Horizontal -> Diode_SMD:D_SOD-123
- SW1: footprint Button_Switch_SMD:SW_Push_1P1T_NO_6x6mm_H9.5mm -> random-keyboard-parts:SKQG-1155865
- moved D17 4.03 mm to (177.0, 146.0)
- moved D14 4.03 mm to (196.1, 127.0)
- moved D6 4.03 mm to (196.1, 88.9)
- moved D11 4.03 mm to (138.9, 127.0)
- moved D12 4.03 mm to (158.0, 127.0)
- moved D13 4.03 mm to (177.0, 127.0)
- moved D3 4.03 mm to (138.9, 88.9)
- moved D4 4.03 mm to (158.0, 88.9)
- moved D5 4.03 mm to (177.0, 88.9)
- moved D1 4.03 mm to (138.9, 60.3)
- moved D2 4.03 mm to (158.0, 60.3)
- moved D10 4.03 mm to (196.1, 107.9)
- moved D18 4.03 mm to (196.1, 146.0)
- moved D15 4.03 mm to (138.9, 146.0)
- moved D16 4.03 mm to (158.0, 146.0)
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Routing:
- net Net-(R1-Pad2): track 27.8 -> 17.9 mm
- net ROW1: track 79.2 -> 86.9 mm, vias 0 -> 1
- net ROW2: track 98.8 -> 105.7 mm, vias 0 -> 1
- net ROW3: track 118.9 -> 125.0 mm, vias 0 -> 1
- net ROW4: track 139.1 -> 144.5 mm, vias 0 -> 1
- net ROW0: track 50.0 -> 54.7 mm, vias 0 -> 1
- net Net-(D14-Pad2): track 6.31 -> 8.47 mm
- net Net-(D6-Pad2): track 6.31 -> 8.47 mm
- net Net-(D10-Pad2): track 6.31 -> 8.47 mm
- net Net-(D18-Pad2): track 6.31 -> 8.47 mm
- net Net-(D2-Pad2): track 6.31 -> 8.47 mm
- net Net-(D1-Pad2): track 6.31 -> 8.47 mm
- net Net-(D5-Pad2): track 6.31 -> 8.47 mm
- net Net-(D13-Pad2): track 6.31 -> 8.47 mm
- net Net-(D12-Pad2): track 6.31 -> 8.47 mm
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
Commit message: Generated gerbers
Parts:
- added H1: MountingHole_2.2mm_M2, MountingHole:MountingHole_2.2mm_M2, F.Cu at (121.4, 74.6)
- added H2: MountingHole_2.2mm_M2, MountingHole:MountingHole_2.2mm_M2, F.Cu at (196.1, 74.6)
- added H3: MountingHole_2.2mm_M2, MountingHole:MountingHole_2.2mm_M2, F.Cu at (121.4, 136.5)
- added H4: MountingHole_2.2mm_M2, MountingHole:MountingHole_2.2mm_M2, F.Cu at (196.1, 136.5)
Other:
- board size 77.8 x 110.3 mm -> 82.6 x 109.5 mm
- board text added: "\///\//\ `/"
- board text removed: "\///\//\`/"
Changed lines of the file:
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@@
     (tracks 400)
     (zones 0)
-    (modules 56)
+    (modules 60)
     (nets 61)
   )
@@
     (visible_elements 7FFFFFFF)
     (pcbplotparams
-      (layerselection 0x010fc_ffffffff)
-      (usegerberextensions false)
+      (layerselection 0x010f0_ffffffff)
+      (usegerberextensions true)
       (usegerberattributes false)
       (usegerberadvancedattributes false)
@@
       (plotinvisibletext false)
       (padsonsilk false)
-      (subtractmaskfromsilk false)
+      (subtractmaskfromsilk true)
       (outputformat 1)
       (mirror false)
-      (drillshape 1)
+      (drillshape 0)
       (scaleselection 1)
-      (outputdirectory ""))
+      (outputdirectory "../Gerbers/"))
   )
   (net 0 "")
@@
     (add_net VCC)
   )
+  (module MountingHole:MountingHole_2.2mm_M2 (layer F.Cu)
+    (at 196.05625 74.6125)
+    (descr "Mounting Hole 2.2mm, no annular, M2")
+    (tags "mounting hole 2.2mm no annular m2")
+    (attr virtual)
+    (fp_text reference H2 (at 0 -3.2) (layer F.SilkS) hide
+      (effects (font (size 1 1) (thickness 0.15)))
+    )
+    (fp_text value MountingHole_2.2mm_M2 (at 11.11377 0.00127) (layer F.Fab)
+      (effects (font (size 1 1) (thickness 0.15)))
+    )
+    (fp_text user %R (at 0.3 0) (layer F.Fab)
+      (effects (font (size 1 1) (thickness 0.15)))
+    )
+    (fp_circle (center 0 0) (end 2.2 0) (layer Cmts.User) (width 0.15))
+    (fp_circle (center 0 0) (end 2.45 0) (layer F.CrtYd) (width 0.05))
+    (pad 1 np_thru_hole circle (at 0 0) (size 2.2 2.2) (drill 2.2) (layers *.Cu *.Mask))
+  )
+  (module MountingHole:MountingHole_2.2mm_M2 (layer F.Cu)
+    (at 121.44375 74.6125)
+    (descr "Mounting Hole 2.2mm, no annular, M2")
+    (tags "mounting hole 2.2mm no annular m2")
+    (attr virtual)
+    (fp_text reference H1 (at 0 -3.2) (layer F.SilkS) hide
+      (effects (font (size 1 1) (thickness 0.15)))
+    )
+    (fp_text value MountingHole_2.2mm_M2 (at -10.31875 0) (layer F.Fab)
+      (effects (font (size 1 1) (thickness 0.15)))
+    )
+    (fp_text user %R (at 0.3 0) (layer F.Fab)
+      (effects (font (size 1 1) (thickness 0.15)))
+    )
+    (fp_circle (center 0 0) (end 2.2 0) (layer Cmts.User) (width 0.15))
+    (fp_circle (center 0 0) (end 2.45 0) (layer F.CrtYd) (width 0.05))
+    (pad 1 np_thru_hole circle (at 0 0) (size 2.2 2.2) (drill 2.2) (layers *.Cu *.Mask))
+  )
+  (module MountingHole:MountingHole_2.2mm_M2 (layer F.Cu)
+    (at 121.44375 136.525)
+    (descr "Mounting Hole 2.2mm, no annular, M2")
+    (tags "mounting hole 2.2mm no annular m2")
+    (attr virtual)
+    (fp_text reference H3 (at 0 -3.2) (layer F.SilkS) hide
+      (effects (font (size 1 1) (thickness 0.15)))
+    )
+    (fp_text value MountingHole_2.2mm_M2 (at -10.31748 0.00127) (layer F.Fab)
+      (effects (font (size 1 1) (thickness 0.15)))
+    )
+    (fp_text user %R (at 0.3 0) (layer F.Fab)
+      (effects (font (size 1 1) (thickness 0.15)))
+    )
+    (fp_circle (center 0 0) (end 2.2 0) (layer Cmts.User) (width 0.15))
+    (fp_circle (center 0 0) (end 2.45 0) (layer F.CrtYd) (width 0.05))
+    (pad 1 np_thru_hole circle (at 0 0) (size 2.2 2.2) (drill 2.2) (layers *.Cu *.Mask))
+  )
+  (module MountingHole:MountingHole_2.2mm_M2 (layer F.Cu)
+    (at 196.05625 136.525)
+    (descr "Mounting Hole 2.2mm, no annular, M2")
+    (tags "mounting hole 2.2mm no annular m2")
+    (attr virtual)
+    (fp_text reference H4 (at 0 -3.2) (layer F.SilkS) hide
+      (effects (font (size 1 1) (thickness 0.15)))
+    )
+    (fp_text value MountingHole_2.2mm_M2 (at 11.1125 0) (layer F.Fab)
+      (effects (font (size 1 1) (thickness 0.15)))
+    )
+    (fp_circle (center 0 0) (end 2.45 0) (layer F.CrtYd) (width 0.05))
+    (fp_circle (center 0 0) (end 2.2 0) (layer Cmts.User) (width 0.15))
+    (fp_text user %R (at 0.3 0) (layer F.Fab)
+      (effects (font (size 1 1) (thickness 0.15)))
+    )
+    (pad 1 np_thru_hole circle (at 0 0) (size 2.2 2.2) (drill 2.2) (layers *.Cu *.Mask))
+  )
   (module random-keyboard-parts:SKQG-1155865 (layer F.Cu)
     (at 165.1 51.435 180)
@@
     (tags SOD-123)
     (attr smd)
-    (fp_text reference D18 (at 3.93827 -0.00127 90) (layer B.SilkS)
+    (fp_text reference D18 (at -0.03048 2.37998 90) (layer B.SilkS)
       (effects (font (size 1 1) (thickness 0.15)) (justify mirror))
     )
@@
     (fp_line (start 0.25 0) (end 0.75 0) (layer B.Fab) (width 0.1))
     (fp_line (start -2.25 1) (end -2.25 -1) (layer B.SilkS) (width 0.12))
-    (fp_text user %R (at 3.93827 -0.00127 90) (layer B.Fab)
+    (fp_text user %R (at -0.03048 2.37998 90) (layer B.Fab)
       (effects (font (size 1 1) (thickness 0.15)) (justify mirror))
     )
@@
     (tags SOD-123)
     (attr smd)
-    (fp_text reference D14 (at 3.93827 -0.00127 90) (layer B.SilkS)
+    (fp_text reference D14 (at -0.03048 2.37998 90) (layer B.SilkS)
       (effects (font (size 1 1) (thickness 0.15)) (justify mirror))
     )
@@
     (fp_line (start 0.25 0) (end 0.75 0) (layer B.Fab) (width 0.1))
     (fp_line (start -2.25 1) (end -2.25 -1) (layer B.SilkS) (width 0.12))
-    (fp_text user %R (at 3.93827 -0.00127 90) (layer B.Fab)
+    (fp_text user %R (at -0.03048 2.37998 90) (layer B.Fab)
       (effects (font (size 1 1) (thickness 0.15)) (justify mirror))
     )
@@
     (tags SOD-123)
     (attr smd)
-    (fp_text reference D10 (at 3.93827 -0.00127 90) (layer B.SilkS)
+    (fp_text reference D10 (at -0.03048 2.37998 90) (layer B.SilkS)
       (effects (font (size 1 1) (thickness 0.15)) (justify mirror))
     )
@@
     (fp_line (start 0.25 0) (end 0.75 0) (layer B.Fab) (width 0.1))
     (fp_line (start -2.25 1) (end -2.25 -1) (layer B.SilkS) (width 0.12))
-    (fp_text user %R (at 3.93827 -0.00127 90) (layer B.Fab)
+    (fp_text user %R (at -0.03048 2.37998 90) (layer B.Fab)
       (effects (font (size 1 1) (thickness 0.15)) (justify mirror))
     )
@@
     (tags SOD-123)
     (attr smd)
-    (fp_text reference D6 (at 3.93827 -0.00127 90) (layer B.SilkS)
+    (fp_text reference D6 (at -0.03048 2.37998 90) (layer B.SilkS)
       (effects (font (size 1 1) (thickness 0.15)) (justify mirror))
     )
@@
     (fp_line (start 0.25 0) (end 0.75 0) (layer B.Fab) (width 0.1))
     (fp_line (start -2.25 1) (end -2.25 -1) (layer B.SilkS) (width 0.12))
-    (fp_text user %R (at 3.93827 -0.00127 90) (layer B.Fab)
+    (fp_text user %R (at -0.03048 2.37998 90) (layer B.Fab)
       (effects (font (size 1 1) (thickness 0.15)) (justify mirror))
     )
@@
     )
   )
-  (gr_arc (start 193.675 152.4) (end 193.675 156.36875) (angle -89.98167122) (layer Edge.Cuts) (width 0.05))
-  (gr_text \///\//\`/ (at 136.017 74.549) (layer F.Mask)
+  (gr_arc (start 121.44375 151.60625) (end 117.475 151.60625) (angle -90) (layer Edge.Cuts) (width 0.05))
+  (gr_arc (start 196.05625 151.60625) (end 196.05625 155.575) (angle -90) (layer Edge.Cuts) (width 0.05))
+  (gr_arc (start 121.44375 50.00625) (end 121.44375 46.0375) (angle -90) (layer Edge.Cuts) (width 0.05))
+  (gr_arc (start 196.05625 50.00625) (end 200.025 50.00625) (angle -90) (layer Edge.Cuts) (width 0.05))
+  (gr_text "\\///\\//\\ `/" (at 140.7795 48.35525) (layer F.Mask)
     (effects (font (size 2 2) (thickness 0.35)))
   )
-  (gr_text \///\//\`/ (at 136.017 74.549) (layer F.Cu)
+  (gr_text "\\///\\//\\ `/" (at 140.7795 48.35525) (layer F.Cu)
     (effects (font (size 2 2) (thickness 0.35)))
   )
-  (gr_arc (start 193.675 50.00625) (end 197.64375 50.00625) (angle -89.98165948) (layer Edge.Cuts) (width 0.05))
-  (gr_arc (start 123.82627 152.40127) (end 119.85752 152.40127) (angle -90) (layer Edge.Cuts) (width 0.05))
-  (gr_arc (start 123.82627 50.00752) (end 123.82627 46.03877) (angle -90) (layer Edge.Cuts) (width 0.05))
-  (gr_line (start 197.64502 50.00752) (end 197.64502 152.40127) (layer Edge.Cuts) (width 0.05))
-  (gr_line (start 123.82627 46.03877) (end 193.67627 46.03877) (layer Edge.Cuts) (width 0.05))
-  (gr_line (start 119.85752 152.40127) (end 119.85752 50.00752) (layer Edge.Cuts) (width 0.05))
-  (gr_line (start 193.67627 156.37002) (end 123.82627 156.37002) (layer Edge.Cuts) (width 0.05))
+  (gr_line (start 200.025 50.00625) (end 200.025 151.60625) (layer Edge.Cuts) (width 0.05))
+  (gr_line (start 121.44375 46.0375) (end 196.05625 46.0375) (layer Edge.Cuts) (width 0.05))
+  (gr_line (start 117.475 151.60625) (end 117.475 50.00625) (layer Edge.Cuts) (width 0.05))
+  (gr_line (start 196.05625 155.575) (end 121.44375 155.575) (layer Edge.Cuts) (width 0.05))
   (segment (start 189.17002 70.67002) (end 186.67627 70.67002) (width 0.381) (layer F.Cu) (net 1))
   (segment (start 189.70752 71.20752) (end 189.17002 70.67002) (width 0.381) (layer F.Cu) (net 1))

Commit message: Updated Gerbers & increased width on LED
Parts:
- removed H1, H2, H3, H4: MountingHole_2.2mm_M2, MountingHole:MountingHole_2.2mm_M2
- D19: footprint LED_THT:LED_D5.0mm-4_RGB -> rootpad:LED_D5.0mm-4_RGB_spaced
- moved SW1 1.02 mm to (166.1, 51.4)
- moved D19 0.83 mm to (178.1, 51.6)
Routing:
- net Net-(D19-Pad4): track 13.9 -> 16.3 mm
- net Net-(D19-Pad3): track 10.4 -> 12.3 mm
- net Net-(D19-Pad1): track 5.18 -> 6.26 mm
- net Net-(R1-Pad2): track 17.9 -> 16.9 mm
- net GND: track 150.3 -> 151.3 mm
- net +5V: track 98.5 -> 97.6 mm

Commit message: Minor adjustments I think
Parts:
- added REF**: MountingHole_2.2mm_M2, MountingHole:MountingHole_2.2mm_M2, F.Cu at (121.4, 136.5)
- added REF**: MountingHole_2.2mm_M2, MountingHole:MountingHole_2.2mm_M2, F.Cu at (196.1, 136.5)
- added REF**: MountingHole_2.2mm_M2, MountingHole:MountingHole_2.2mm_M2, F.Cu at (196.1, 74.6)
- added REF**: MountingHole_2.2mm_M2, MountingHole:MountingHole_2.2mm_M2, F.Cu at (121.4, 74.6)
Routing:
- net COL1: vias 1 -> 3
Changed lines of the file:
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@@
     (thickness 1.6)
     (drawings 10)
-    (tracks 397)
+    (tracks 403)
     (zones 0)
-    (modules 56)
+    (modules 60)
     (nets 61)
   )
@@
     (add_net VCC)
   )
+  (module MountingHole:MountingHole_2.2mm_M2 (layer F.Cu)
+    (at 121.44375 136.525)
+    (descr "Mounting Hole 2.2mm, no annular, M2")
+    (tags "mounting hole 2.2mm no annular m2")
+    (attr virtual)
+    (fp_text reference REF** (at 0 -3.2) (layer F.SilkS) hide
+      (effects (font (size 1 1) (thickness 0.15)))
+    )
+    (fp_text value MountingHole_2.2mm_M2 (at -11.90625 0) (layer F.Fab)
+      (effects (font (size 1 1) (thickness 0.15)))
+    )
+    (fp_text user %R (at 0.3 0) (layer F.Fab)
+      (effects (font (size 1 1) (thickness 0.15)))
+    )
+    (fp_circle (center 0 0) (end 2.2 0) (layer Cmts.User) (width 0.15))
+    (fp_circle (center 0 0) (end 2.45 0) (layer F.CrtYd) (width 0.05))
+    (pad 1 np_thru_hole circle (at 0 0) (size 2.2 2.2) (drill 2.2) (layers *.Cu *.Mask))
+  )
+  (module MountingHole:MountingHole_2.2mm_M2 (layer F.Cu)
+    (at 196.05625 136.525)
+    (descr "Mounting Hole 2.2mm, no annular, M2")
+    (tags "mounting hole 2.2mm no annular m2")
+    (attr virtual)
+    (fp_text reference REF** (at 0 -3.2) (layer F.SilkS) hide
+      (effects (font (size 1 1) (thickness 0.15)))
+    )
+    (fp_text value MountingHole_2.2mm_M2 (at 11.90625 0) (layer F.Fab)
+      (effects (font (size 1 1) (thickness 0.15)))
+    )
+    (fp_text user %R (at 0.3 0) (layer F.Fab)
+      (effects (font (size 1 1) (thickness 0.15)))
+    )
+    (fp_circle (center 0 0) (end 2.2 0) (layer Cmts.User) (width 0.15))
+    (fp_circle (center 0 0) (end 2.45 0) (layer F.CrtYd) (width 0.05))
+    (pad 1 np_thru_hole circle (at 0 0) (size 2.2 2.2) (drill 2.2) (layers *.Cu *.Mask))
+  )
+  (module MountingHole:MountingHole_2.2mm_M2 (layer F.Cu)
+    (at 196.05625 74.6125)
+    (descr "Mounting Hole 2.2mm, no annular, M2")
+    (tags "mounting hole 2.2mm no annular m2")
+    (attr virtual)
+    (fp_text reference REF** (at 0 -3.2) (layer F.SilkS) hide
+      (effects (font (size 1 1) (thickness 0.15)))
+    )
+    (fp_text value MountingHole_2.2mm_M2 (at 11.90625 0) (layer F.Fab)
+      (effects (font (size 1 1) (thickness 0.15)))
+    )
+    (fp_circle (center 0 0) (end 2.45 0) (layer F.CrtYd) (width 0.05))
+    (fp_circle (center 0 0) (end 2.2 0) (layer Cmts.User) (width 0.15))
+    (fp_text user %R (at 0.3 0) (layer F.Fab)
+      (effects (font (size 1 1) (thickness 0.15)))
+    )
+    (pad 1 np_thru_hole circle (at 0 0) (size 2.2 2.2) (drill 2.2) (layers *.Cu *.Mask))
+  )
+  (module MountingHole:MountingHole_2.2mm_M2 (layer F.Cu)
+    (at 121.44375 74.6125)
+    (descr "Mounting Hole 2.2mm, no annular, M2")
+    (tags "mounting hole 2.2mm no annular m2")
+    (attr virtual)
+    (fp_text reference REF** (at 0 -3.2) (layer F.SilkS) hide
+      (effects (font (size 1 1) (thickness 0.15)))
+    )
+    (fp_text value MountingHole_2.2mm_M2 (at -11.90625 0) (layer F.Fab)
+      (effects (font (size 1 1) (thickness 0.15)))
+    )
+    (fp_circle (center 0 0) (end 2.45 0) (layer F.CrtYd) (width 0.05))
+    (fp_circle (center 0 0) (end 2.2 0) (layer Cmts.User) (width 0.15))
+    (fp_text user %R (at 0.3 0) (layer F.Fab)
+      (effects (font (size 1 1) (thickness 0.15)))
+    )
+    (pad 1 np_thru_hole circle (at 0 0) (size 2.2 2.2) (drill 2.2) (layers *.Cu *.Mask))
+  )
   (module rootpad:LED_D5.0mm-4_RGB_spaced (layer F.Cu)
     (at 178.1175 51.562)
@@
   (gr_arc (start 121.44375 50.00625) (end 121.44375 46.0375) (angle -90) (layer Edge.Cuts) (width 0.05))
   (gr_arc (start 196.05625 50.00625) (end 200.025 50.00625) (angle -90) (layer Edge.Cuts) (width 0.05))
-  (gr_text "\\///\\//\\ `/" (at 136.0805 74.295) (layer F.Mask)
+  (gr_text "\\///\\//\\ `/" (at 139.7 73.81875) (layer F.Mask)
     (effects (font (size 1.9 1.9) (thickness 0.35)))
   )
-  (gr_text "\\///\\//\\ `/" (at 136.0805 74.295) (layer F.Cu)
+  (gr_text "\\///\\//\\ `/" (at 139.7 73.81875) (layer F.Cu)
     (effects (font (size 1.9 1.9) (thickness 0.35)))
   )
@@
   (segment (start 131.76504 80.9625) (end 126.36627 86.36127) (width 0.254) (layer B.Cu) (net 31))
   (segment (start 168.275 80.9625) (end 131.76504 80.9625) (width 0.254) (layer B.Cu) (net 31))
-  (segment (start 126.36627 59.37726) (end 126.36627 86.36127) (width 0.254) (layer F.Cu) (net 31))
-  (segment (start 126.36627 57.78627) (end 126.36627 59.37726) (width 0.254) (layer F.Cu) (net 31))
+  (segment (start 126.36627 57.78627) (end 126.36627 86.36127) (width 0.254) (layer B.Cu) (net 31))
   (segment (start 145.41627 143.51127) (end 145.41627 124.46127) (width 0.254) (layer F.Cu) (net 32))
   (segment (start 145.41627 105.41127) (end 145.41627 124.46127) (width 0.254) (layer F.Cu) (net 32))
   (segment (start 145.41627 105.41127) (end 145.41627 86.36127) (width 0.254) (layer F.Cu) (net 32))
-  (segment (start 145.41627 57.78627) (end 145.41627 86.36127) (width 0.254) (layer F.Cu) (net 32))
   (via (at 172.24375 75.40625) (size 0.8) (drill 0.4) (layers F.Cu B.Cu) (net 32))
   (segment (start 172.24375 72.69854) (end 172.24375 75.40625) (width 0.254) (layer F.Cu) (net 32))
@@
   (segment (start 150.02129 81.75625) (end 145.41627 86.36127) (width 0.254) (layer B.Cu) (net 32))
   (segment (start 168.275 81.75625) (end 150.02129 81.75625) (width 0.254) (layer B.Cu) (net 32))
+  (segment (start 145.41627 57.78627) (end 145.41627 65.40373) (width 0.254) (layer F.Cu) (net 32))
+  (segment (start 145.41627 65.40373) (end 145.415 65.405) (width 0.254) (layer F.Cu) (net 32))
+  (segment (start 145.415 86.36) (end 145.41627 86.36127) (width 0.254) (layer F.Cu) (net 32))
+  (via (at 145.415 65.405) (size 0.8) (drill 0.4) (layers F.Cu B.Cu) (net 32))
+  (via (at 145.415 80.01) (size 0.8) (drill 0.4) (layers F.Cu B.Cu) (net 32))
+  (segment (start 145.41627 86.36127) (end 145.41627 80.01127) (width 0.254) (layer F.Cu) (net 32))
+  (segment (start 145.41627 80.01127) (end 145.415 80.01) (width 0.254) (layer F.Cu) (net 32))
+  (segment (start 145.415 80.01) (end 145.415 65.405) (width 0.254) (layer B.Cu) (net 32))
   (segment (start 164.46627 124.46127) (end 164.46627 143.51127) (width 0.254) (layer F.Cu) (net 33))
   (via (at 173.0375 74.6125) (size 0.8) (drill 0.4) (layers F.Cu B.Cu) (net 33))
